File: water-meter-counter.kicad_pcb (KiCad board)
At the start: 2 copper layers, 62.8 x 38.4 mm, 42 parts, among them J1 Conn_01x04, J2 Conn_PIC_ICSP_ICD, J3 Conn_01x01, J4 Conn_01x01, U1 PIC18F25K80_IML, U2 HCPL-817-30DE

Commit message: First draft of firmware
Parts:
- removed kibuzzard-6924F154: G***, kibuzzard-6924F154
- removed kibuzzard-6924F163: G***, kibuzzard-6924F163
- added kibuzzard-69451647: G***, kibuzzard-69451647, F.Cu at (163.8, 99.4)
- added kibuzzard-6945164F: G***, kibuzzard-6945164F, F.Cu at (163.8, 98.3)
- moved REF** 23.9 mm to (132.2, 89.8)
- moved REF** 11.0 mm to (131.4, 96.5)
Other:
- board text added: "https://github.com/usimd/water-meter-counter, Rev ${Revision}"

Commit message: Prepare Rev2
Parts:
- removed the REF** at (136.0, 112.3)
- removed the REF** at (134.6, 105.1)
- removed the REF** at (132.2, 89.8)
- removed the REF** at (131.4, 96.5)
- removed kibuzzard-6924F19F: G***, kibuzzard-6924F19F
- removed kibuzzard-6924F1AD: G***, kibuzzard-6924F1AD
- removed kibuzzard-6924F218: G***, kibuzzard-6924F218
- removed kibuzzard-6924F221: G***, kibuzzard-6924F221
- added FID1: Fiducial, Fiducial:Fiducial_1mm_Mask3mm, F.Cu at (128.4, 85.8)
- added FID2: Fiducial, Fiducial:Fiducial_1mm_Mask3mm, F.Cu at (134.0, 114.7)
- added FID3: Fiducial, Fiducial:Fiducial_1mm_Mask3mm, F.Cu at (164.9, 114.8)
- added R4: 330k, Resistor_SMD:R_0603_1608Metric, F.Cu at (140.8, 107.9)
- added R8: 330k, Resistor_SMD:R_0603_1608Metric, F.Cu at (142.5, 107.9)
- added R9: 330k, Resistor_SMD:R_0603_1608Metric, F.Cu at (149.5, 98.3)
- added REF**: OSHW-Symbol_6.7x6mm_SilkScreen, Symbol:OSHW-Symbol_6.7x6mm_SilkScreen, B.Cu at (134.8, 110.2)
- added REF**: KiCad-Logo2_6mm_SilkScreen, Symbol:KiCad-Logo2_6mm_SilkScreen, B.Cu at (164.0, 107.6)
- added kibuzzard-69E7705E: G***, kibuzzard-69E7705E, F.Cu at (146.3, 111.1)
- added kibuzzard-69E77065: G***, kibuzzard-69E77065, F.Cu at (148.8, 111.1)
- added kibuzzard-69E7706B: G***, kibuzzard-69E7706B, F.Cu at (151.3, 111.1)
- added kibuzzard-69E77073: G***, kibuzzard-69E77073, F.Cu at (153.8, 111.1)
- C1, C7: footprint Capacitor_SMD:C_0402_1005Metric_Pad0.74x0.62mm_HandSolder -> Capacitor_SMD:C_0603_1608Metric
- C2: footprint Capacitor_SMD:C_0402_1005Metric_Pad0.74x0.62mm_HandSolder -> Capacitor_SMD:C_0603_1608Metric; moved to B.Cu
- C3: value 0.1uF -> 10uF; footprint Capacitor_SMD:C_0402_1005Metric_Pad0.74x0.62mm_HandSolder -> Capacitor_SMD:C_0603_1608Metric
- C4: footprint Capacitor_SMD:C_0603_1608Metric_Pad1.08x0.95mm_HandSolder -> Capacitor_SMD:C_0603_1608Metric
- C5: renamed from C6; footprint Capacitor_SMD:C_0603_1608Metric_Pad1.08x0.95mm_HandSolder -> Capacitor_SMD:C_0603_1608Metric
- C6: renamed from C5; footprint Capacitor_SMD:C_0402_1005Metric_Pad0.74x0.62mm_HandSolder -> Capacitor_SMD:C_0603_1608Metric
- J2: footprint Connector_PinHeader_1.00mm:PinHeader_1x06_P1.00mm_Vertical -> Connector_PinHeader_1.27mm:PinHeader_1x06_P1.27mm_Vertical
- L1, L2: value 1mH -> 470uH
- R1, R2, R7: footprint Resistor_SMD:R_0402_1005Metric_Pad0.72x0.64mm_HandSolder -> Resistor_SMD:R_0603_1608Metric
- R10: renamed from R4; footprint Resistor_SMD:R_0402_1005Metric_Pad0.72x0.64mm_HandSolder -> Resistor_SMD:R_0603_1608Metric
- R11: renamed from R8; footprint Resistor_SMD:R_0402_1005Metric_Pad0.72x0.64mm_HandSolder -> Resistor_SMD:R_0603_1608Metric
- R3: renamed from R6; footprint Resistor_SMD:R_0805_2012Metric_Pad1.20x1.40mm_HandSolder -> Resistor_SMD:R_0805_2012Metric
- R5: value 220 -> 330k; footprint Resistor_SMD:R_0805_2012Metric_Pad1.20x1.40mm_HandSolder -> Resistor_SMD:R_0603_1608Metric
- R6: renamed from R3; footprint Resistor_SMD:R_0402_1005Metric_Pad0.72x0.64mm_HandSolder -> Resistor_SMD:R_0603_1608Metric
- moved R3 31.2 mm to (171.6, 109.1), turned to -90 degrees
- moved U2 17.2 mm to (164.6, 109.1), turned to 180 degrees
- moved C2 15.5 mm to (146.1, 106.1), turned to 135 degrees
- moved R2 12.8 mm to (151.6, 107.1), turned to 135 degrees
- moved R5 11.9 mm to (148.7, 96.7), turned to 180 degrees
- moved C6 11.5 mm to (133.9, 104.6), turned to 180 degrees
- moved R6 11.1 mm to (138.5, 107.1)
- moved C4 11.0 mm to (135.5, 107.1)
- moved R1 10.6 mm to (153.8, 104.9), turned to -45 degrees
- moved L2 10.5 mm to (138.8, 94.6), turned to 120 degrees
- moved C1 10.4 mm to (152.7, 106.0), turned to -45 degrees
- moved D2 9.56 mm to (138.9, 104.9)
- moved U1 8.92 mm to (147.4, 104.0), turned to -135 degrees
- moved R10 7.36 mm to (142.4, 102.8), turned to -135 degrees
- moved kibuzzard-6924F10E 6.75 mm to (158.1, 99.8), turned to -90 degrees
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- renumbered D2 to D1, D1 to D2, H2 to H1, H3 to H2, H1 to H3
Connections:
- net Net-(D1-K) renamed /TANK_A
- net Net-(D3-K) renamed /TANK_B
- C3 pad 1: +5V -> GND
- C3 pad 2: GND -> Net-(U1-Vcap)
- R5 pad 1: Net-(R5-Pad1) -> +5V
- R5 pad 2: /S0_P -> /PULSE_B
- U1 pad 20: /S0_PULSE_OUT -> unconnected-(U1-CANTX/INT2/RB2-Pad20)
- U1 pad 22: unconnected-(U1-AN9/ECCP1/RB4-Pad22) -> /S0_PULSE_OUT
- U1 pad 3: +5V -> Net-(U1-Vcap)
- U2 pad 4: Net-(R5-Pad1) -> /S0_P
Routing:
- net GND: track 10.5 -> 69.5 mm, vias 9 -> 13
- net +5V: track 44.8 -> 65.3 mm, vias 1 -> 6
- net /ICSPCLK: track 4.59 -> 21.8 mm
- net /ICSPDAT: track 4.45 -> 20.1 mm
- net /TANK_B: track 20.3 -> 9.33 mm
- net /~{MCLR}: track 5.38 -> 12.9 mm
- net /RX: track 26.7 -> 33.4 mm, vias 2 -> 1
- net /S0_PULSE_OUT: track 16.7 -> 23.1 mm
- net /TX: track 23.9 -> 29.6 mm
- net /TANK_A: track 13.2 -> 9.27 mm
- net /PULSE_A: track 9.85 -> 7.00 mm
- net Net-(U1-Vcap): track 0.00 -> 2.26 mm
- net Net-(R5-Pad1): track 2.20 -> 0.00 mm
- net /PULSE_B: track 5.93 -> 7.91 mm
- net /S0_N: track 7.31 -> 5.56 mm
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