File: water-meter-counter.kicad_pcb (KiCad board)
At the start: 2 copper layers, 62.8 x 38.4 mm, 46 parts, among them J1 Conn_01x04, J2 Conn_PIC_ICSP_ICD, J3 Conn_01x01, J4 Conn_01x01, U1 PIC18F25K80_IML, U2 HCPL-817-30DE

Commit message: Rev2 firmware, release CI and licensing
Firmware:
- Comparator-only ring-down sensing on both LC tanks (Timer1 gated by
  comparator 1 against CVREF), no ADC.
- New hardware-independent rotation decoder (B pass detection, direction
  from A's first vs. last third of the pass).
- Sleep between samples with WDT wake-up, S0 pulse timed by TMR0.
- DEBUG_STREAM selectable by the build; user.cmake builds a second
  default-debug image next to the production one.
- Commit the MPLAB-generated CMake files so CI can build; pack path
  defaults to $HOME/.mchp_packs.

CI:
- Fix firmware build (preset, XC8 from setup-xc-action).
- Hardware job on KiCad 10: ERC/DRC reports, schematic PDF, BOM,
  pick-and-place, Gerbers and drill files.
- REUSE compliance check.
- Release job for v* tags bundling firmware, hardware, housing and
  license texts.

Licensing:
- REUSE layout: hardware CERN-OHL-S-2.0, firmware Apache-2.0,
  MCC-generated drivers under Microchip's terms.

Co-authored-by: Copilot <223556219+Copilot@users.noreply.github.com>
Parts:
- renumbered REF** to LOGO1, REF** to LOGO2
