File: water-meter-counter.kicad_sch (KiCad schematic)
At the start: 29 parts, among them J1 Conn_01x04, J2 Conn_PIC_ICSP_ICD, J3 Conn_01x01, J4 Conn_01x01, U1 PIC18F25K80_IML, U2 HCPL-817-30DE

Commit message: First draft of firmware
Parts:
- J2: now left out of the parts list
Other:
- title: (none) -> Water meter counter
Changed lines of the file:
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@@
 	(generator_version "9.0")
 	(paper "A5")
+	(title_block
+		(title "Water meter counter")
+		(rev "${Revision}")
+		(comment 3 "Inductive water meter counter with S0 interface for GSB-8 style meters")
+	)
 	(rectangle
 		(start 45.72 13.97)
@@
 		(unit 1)
 		(exclude_from_sim no)
-		(in_bom yes)
+		(in_bom no)
 		(on_board yes)
 		(dnp no)

Commit message: Prepare Rev2
Parts:
- removed C3: 0.1uF, Capacitor_SMD:C_0402_1005Metric_Pad0.74x0.62mm_HandSolder, symbol Device:C
- removed R5: 220, Resistor_SMD:R_0805_2012Metric_Pad1.20x1.40mm_HandSolder, symbol Device:R
- added C3: 10uF, Capacitor_SMD:C_0603_1608Metric, symbol Device:C_Small
- added FID1, FID2, FID3: Fiducial, Fiducial:Fiducial_1mm_Mask3mm, symbol Mechanical:Fiducial
- added R4, R5, R8, R9: 330k, Resistor_SMD:R_0603_1608Metric, symbol Device:R_Small
- C1, C2: footprint Capacitor_SMD:C_0402_1005Metric_Pad0.74x0.62mm_HandSolder -> Capacitor_SMD:C_0603_1608Metric; symbol Device:C -> Device:C_Small
- C4: footprint Capacitor_SMD:C_0603_1608Metric_Pad1.08x0.95mm_HandSolder -> Capacitor_SMD:C_0603_1608Metric
- C5: renamed from C6; footprint Capacitor_SMD:C_0603_1608Metric_Pad1.08x0.95mm_HandSolder -> Capacitor_SMD:C_0603_1608Metric
- C6: renamed from C5; footprint Capacitor_SMD:C_0402_1005Metric_Pad0.74x0.62mm_HandSolder -> Capacitor_SMD:C_0603_1608Metric
- C7: footprint Capacitor_SMD:C_0402_1005Metric_Pad0.74x0.62mm_HandSolder -> Capacitor_SMD:C_0603_1608Metric
- D2: renamed from D1; MPN (none) -> SD103AW
- D3: MPN (none) -> SD103AW
- J2: footprint Connector_PinHeader_1.00mm:PinHeader_1x06_P1.00mm_Vertical -> Connector_PinHeader_1.27mm:PinHeader_1x06_P1.27mm_Vertical
- L1, L2: value 1mH -> 470uH; MPN 05HCP-102K-51 -> 05HCP-471K-51
- R1, R2, R7: footprint Resistor_SMD:R_0402_1005Metric_Pad0.72x0.64mm_HandSolder -> Resistor_SMD:R_0603_1608Metric
- R10: renamed from R4; footprint Resistor_SMD:R_0402_1005Metric_Pad0.72x0.64mm_HandSolder -> Resistor_SMD:R_0603_1608Metric
- R11: renamed from R8; footprint Resistor_SMD:R_0402_1005Metric_Pad0.72x0.64mm_HandSolder -> Resistor_SMD:R_0603_1608Metric
- R3: renamed from R6; footprint Resistor_SMD:R_0805_2012Metric_Pad1.20x1.40mm_HandSolder -> Resistor_SMD:R_0805_2012Metric
- R6: renamed from R3; footprint Resistor_SMD:R_0402_1005Metric_Pad0.72x0.64mm_HandSolder -> Resistor_SMD:R_0603_1608Metric
- renumbered D2 to D1, H2 to H1, H3 to H2, H1 to H3
Connections:
- net +5V: now also R4.1, R5.1; no longer U1.3 (Vcap)
- net GND: now also C3.1, R8.2, R9.2
- net PULSE_A: now also R4.2, R8.1
- net PULSE_B: now also R5.2, R9.1
- net S0_P: now also U2.4
- net S0_PULSE_OUT: now also U1.22 (AN9/ECCP1/RB4); no longer U1.20 (CANTX/INT2/RB2)
- net TANK_A: now reaches C4.1, C6.1, D2.1 (K), L1.1
- net TANK_B: now reaches C5.1, C7.1, D3.1 (K), L2.1
- new net: C3.2, U1.3 (Vcap)
Other:
- moved on the sheet: C1, C2, C4, C5, C7, D3, H1, H2, H3, R11, R6, R7
