File: water-meter-counter.kicad_sch (KiCad schematic)
At the start: 35 parts, among them J1 Conn_01x04, J2 Conn_PIC_ICSP_ICD, J3 Conn_01x01, J4 Conn_01x01, U1 PIC18F25K80_IML, U2 HCPL-817-30DE

Commit message: Rev2 firmware, release CI and licensing
Firmware:
- Comparator-only ring-down sensing on both LC tanks (Timer1 gated by
  comparator 1 against CVREF), no ADC.
- New hardware-independent rotation decoder (B pass detection, direction
  from A's first vs. last third of the pass).
- Sleep between samples with WDT wake-up, S0 pulse timed by TMR0.
- DEBUG_STREAM selectable by the build; user.cmake builds a second
  default-debug image next to the production one.
- Commit the MPLAB-generated CMake files so CI can build; pack path
  defaults to $HOME/.mchp_packs.

CI:
- Fix firmware build (preset, XC8 from setup-xc-action).
- Hardware job on KiCad 10: ERC/DRC reports, schematic PDF, BOM,
  pick-and-place, Gerbers and drill files.
- REUSE compliance check.
- Release job for v* tags bundling firmware, hardware, housing and
  license texts.

Licensing:
- REUSE layout: hardware CERN-OHL-S-2.0, firmware Apache-2.0,
  MCC-generated drivers under Microchip's terms.

Co-authored-by: Copilot <223556219+Copilot@users.noreply.github.com>
Parts:
- C1: MPN (none) -> 06035C104JAT2A; Manufacturer (none) -> KYOCERA AVX; now not fitted
- C2: MPN (none) -> 06035C104JAT2A; Manufacturer (none) -> KYOCERA AVX
- C3: MPN (none) -> GRM188R61E106KA73D; Manufacturer (none) -> Murata
- C4, C5: MPN (none) -> C0603C101J5GACTU; Manufacturer (none) -> KEMET
- C6, C7: MPN (none) -> C0603C222J5GACTU; Manufacturer (none) -> KEMET
- D1: MPN (none) -> B5819W; Manufacturer (none) -> MDD (Microdiode Semiconductor)
- D2, D3: MPN SD103AW -> SS14MH; Manufacturer (none) -> Taiwan Semiconductor
- J1: MPN (none) -> S4B-XH-A(LF)(SN); Manufacturer (none) -> JST
- L1, L2: Manufacturer (none) -> Fastron
- R1: MPN (none) -> ESR03EZPJ103; Manufacturer (none) -> ROHM
- R10, R11, R2, R6, R7: MPN (none) -> RC0603FR-07470RL; Manufacturer (none) -> YAGEO
- R3: MPN (none) -> RC0805FR-07220RL; Manufacturer (none) -> YAGEO
- R4, R5, R8, R9: MPN (none) -> RC0603FR-07330KL; Manufacturer (none) -> YAGEO
- U1: MPN (none) -> PIC18F25K80-I/MM; Manufacturer (none) -> Microchip
- U2: MPN (none) -> HCPL-817-30DE; Manufacturer (none) -> Broadcom
Other:
- note added: "C1 DNP: No capacitance on MCLR/VPP during ICSP (datasheet + PICkit 5 troubleshooting). Populate if programming fails."
